File: PCB/fate.kicad_pcb (KiCad board)
At the start: 2 copper layers, 125 x 115 mm, 33 parts, among them J1 XLR3, J10 Conn_01x01, J2 Conn_Coaxial, J3 Conn_Coaxial, J4 Conn_Coaxial, J5 Conn_Coaxial, J6 XLR3, J7 Conn_01x01, J8 Conn_01x01, J9 Conn_01x01

Commit message: Add ground reference between differential signal lines
Parts:
- moved R3 25.4 mm to (160.4, 61.0), turned to 180 degrees
- moved R9 25.4 mm to (160.4, 105.0), turned to 180 degrees
- moved H1 11.0 mm to (101.0, 39.0)
- moved H3 11.0 mm to (101.0, 136.0)
Connections:
- R10 pad 1: Net-(R10-Pad1) -> GND
- R3 pad 2: Net-(R3-Pad2) -> GND
- R4 pad 1: Net-(R3-Pad2) -> GND
- R9 pad 2: Net-(R10-Pad1) -> GND
Routing:
- net Net-(R3-Pad2): track 29.5 -> 0.00 mm
- net Net-(R10-Pad1): track 29.5 -> 0.00 mm
- net /OUT_RIGHT+: track 103.5 -> 80.9 mm
- net /OUT_LEFT+: track 106.7 -> 85.2 mm
- net GND: vias 268 -> 267
Other:
- board size 125 x 115 mm -> 130 x 115 mm
- board text added: "FATE - DC20190209"
- board text removed: "FATE - DC20190208"
